File: eagle-boards/trinket-m0/trinket-mcp23017.sch (EAGLE design)
At the start: 8 parts, among them IC2 MCP23017SP, Q1 BC547

Commit message: Clean up the Trinket M0 based boards.
This makes the two board use the same size, and the same positioning of the common components.

It also reorients the silkscreen markings on the back to have the same orientation as the actuator board.

Also mark the used lines from the Trinket, as you can technically use any other MCU that can drive I²C.
Parts:
- renumbered IC2 to IC1
Changed lines of the file:
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@@
 <part name="GND5" library="supply1" library_urn="urn:adsk.eagle:library:371" deviceset="GND" device=""/>
 <part name="R3" library="rcl" library_urn="urn:adsk.eagle:library:334" deviceset="R-EU_" device="0207/10" package3d_urn="urn:adsk.eagle:package:23491/2" value="1k"/>
-<part name="IC2" library="microchip" library_urn="urn:adsk.eagle:library:294" deviceset="MCP23017" device="SP" package3d_urn="urn:adsk.eagle:package:20799/2"/>
+<part name="IC1" library="microchip" library_urn="urn:adsk.eagle:library:294" deviceset="MCP23017" device="SP" package3d_urn="urn:adsk.eagle:package:20799/2"/>
 </parts>
 <sheets>
@@
 <attribute name="VALUE" x="100.33" y="19.558" size="1.778" layer="96"/>
 </instance>
-<instance part="IC2" gate="G$1" x="40.64" y="76.2" smashed="yes">
+<instance part="IC1" gate="G$1" x="40.64" y="76.2" smashed="yes">
 <attribute name="NAME" x="30.48" y="100.33" size="1.778" layer="95"/>
 <attribute name="VALUE" x="30.48" y="50.8" size="1.778" layer="96"/>
@@
 </segment>
 <segment>
-<pinref part="IC2" gate="G$1" pin="A1"/>
+<pinref part="IC1" gate="G$1" pin="A1"/>
 <pinref part="GND4" gate="1" pin="GND"/>
 <wire x1="27.94" y1="63.5" x2="22.86" y2="63.5" width="0.1524" layer="91"/>
 <wire x1="22.86" y1="63.5" x2="22.86" y2="60.96" width="0.1524" layer="91"/>
-<pinref part="IC2" gate="G$1" pin="A2"/>
+<pinref part="IC1" gate="G$1" pin="A2"/>
 <wire x1="22.86" y1="60.96" x2="22.86" y2="55.88" width="0.1524" layer="91"/>
 <wire x1="22.86" y1="55.88" x2="22.86" y2="48.26" width="0.1524" layer="91"/>
 <wire x1="27.94" y1="60.96" x2="22.86" y2="60.96" width="0.1524" layer="91"/>
 <junction x="22.86" y="60.96"/>
-<pinref part="IC2" gate="G$1" pin="VSS"/>
+<pinref part="IC1" gate="G$1" pin="VSS"/>
 <wire x1="27.94" y1="55.88" x2="22.86" y2="55.88" width="0.1524" layer="91"/>
 <junction x="22.86" y="55.88"/>
@@
 </segment>
 <segment>
-<pinref part="IC2" gate="G$1" pin="VDD"/>
+<pinref part="IC1" gate="G$1" pin="VDD"/>
 <wire x1="27.94" y1="96.52" x2="22.86" y2="96.52" width="0.1524" layer="91"/>
 <pinref part="+3V3" gate="G$1" pin="+3V3"/>
@@
 <wire x1="10.16" y1="83.82" x2="10.16" y2="96.52" width="0.1524" layer="91"/>
 <junction x="10.16" y="96.52"/>
-<pinref part="IC2" gate="G$1" pin="!RESET"/>
+<pinref part="IC1" gate="G$1" pin="!RESET"/>
 <wire x1="27.94" y1="91.44" x2="22.86" y2="91.44" width="0.1524" layer="91"/>
 <wire x1="22.86" y1="91.44" x2="22.86" y2="96.52" width="0.1524" layer="91"/>
 <junction x="22.86" y="96.52"/>
-<pinref part="IC2" gate="G$1" pin="A0"/>
+<pinref part="IC1" gate="G$1" pin="A0"/>
 <wire x1="27.94" y1="66.04" x2="22.86" y2="66.04" width="0.1524" layer="91"/>
 <wire x1="22.86" y1="66.04" x2="22.86" y2="91.44" width="0.1524" layer="91"/>
@@
 <wire x1="17.78" y1="73.66" x2="27.94" y2="73.66" width="0.1524" layer="91"/>
 <wire x1="17.78" y1="73.66" x2="17.78" y2="10.16" width="0.1524" layer="91"/>
-<pinref part="IC2" gate="G$1" pin="SCL"/>
+<pinref part="IC1" gate="G$1" pin="SCL"/>
 <pinref part="R1" gate="G$1" pin="1"/>
 <wire x1="17.78" y1="73.66" x2="10.16" y2="73.66" width="0.1524" layer="91"/>
@@
 <junction x="15.24" y="71.12"/>
 <wire x1="15.24" y1="71.12" x2="15.24" y2="-40.64" width="0.1524" layer="91"/>
-<pinref part="IC2" gate="G$1" pin="SDA"/>
+<pinref part="IC1" gate="G$1" pin="SDA"/>
 <pinref part="R2" gate="G$1" pin="1"/>
 <wire x1="15.24" y1="71.12" x2="2.54" y2="71.12" width="0.1524" layer="91"/>
@@
 <pinref part="MCU" gate="A" pin="2"/>
 <wire x1="127" y1="96.52" x2="53.34" y2="96.52" width="0.1524" layer="91"/>
-<pinref part="IC2" gate="G$1" pin="GPA0"/>
+<pinref part="IC1" gate="G$1" pin="GPA0"/>
 </segment>
 </net>
@@
 <pinref part="MCU" gate="A" pin="3"/>
 <wire x1="53.34" y1="93.98" x2="127" y2="93.98" width="0.1524" layer="91"/>
-<pinref part="IC2" gate="G$1" pin="GPA1"/>
+<pinref part="IC1" gate="G$1" pin="GPA1"/>
 </segment>
 </net>
@@
 <pinref part="MCU" gate="A" pin="4"/>
 <wire x1="127" y1="91.44" x2="53.34" y2="91.44" width="0.1524" layer="91"/>
-<pinref part="IC2" gate="G$1" pin="GPA2"/>
+<pinref part="IC1" gate="G$1" pin="GPA2"/>
 </segment>
 </net>
@@
 <pinref part="MCU" gate="A" pin="5"/>
 <wire x1="127" y1="88.9" x2="53.34" y2="88.9" width="0.1524" layer="91"/>
-<pinref part="IC2" gate="G$1" pin="GPA3"/>
+<pinref part="IC1" gate="G$1" pin="GPA3"/>
 </segment>
 </net>
@@
 <pinref part="MCU" gate="A" pin="6"/>
 <wire x1="127" y1="86.36" x2="53.34" y2="86.36" width="0.1524" layer="91"/>
-<pinref part="IC2" gate="G$1" pin="GPA4"/>
+<pinref part="IC1" gate="G$1" pin="GPA4"/>
 </segment>
 </net>
@@
 <pinref part="MCU" gate="A" pin="7"/>
 <wire x1="127" y1="83.82" x2="53.34" y2="83.82" width="0.1524" layer="91"/>
-<pinref part="IC2" gate="G$1" pin="GPA5"/>
+<pinref part="IC1" gate="G$1" pin="GPA5"/>
 </segment>
 </net>
@@
 <pinref part="MCU" gate="A" pin="8"/>
 <wire x1="127" y1="81.28" x2="53.34" y2="81.28" width="0.1524" layer="91"/>
-<pinref part="IC2" gate="G$1" pin="GPA6"/>
+<pinref part="IC1" gate="G$1" pin="GPA6"/>
 </segment>
 </net>
@@
 <pinref part="MCU" gate="A" pin="9"/>
 <wire x1="127" y1="78.74" x2="53.34" y2="78.74" width="0.1524" layer="91"/>
-<pinref part="IC2" gate="G$1" pin="GPA7"/>
+<pinref part="IC1" gate="G$1" pin="GPA7"/>
 </segment>
 </net>
@@
 <segment>
 <pinref part="MCU" gate="A" pin="10"/>
-<pinref part="IC2" gate="G$1" pin="GPB0"/>
+<pinref part="IC1" gate="G$1" pin="GPB0"/>
 <wire x1="53.34" y1="73.66" x2="53.34" y2="76.2" width="0.1524" layer="91"/>
 <wire x1="53.34" y1="76.2" x2="127" y2="76.2" width="0.1524" layer="91"/>
@@
 <segment>
 <pinref part="MCU" gate="A" pin="11"/>
-<pinref part="IC2" gate="G$1" pin="GPB1"/>
+<pinref part="IC1" gate="G$1" pin="GPB1"/>
 <wire x1="53.34" y1="71.12" x2="55.88" y2="71.12" width="0.1524" layer="91"/>
 <wire x1="55.88" y1="71.12" x2="55.88" y2="73.66" width="0.1524" layer="91"/>
@@
 <segment>
 <pinref part="MCU" gate="A" pin="12"/>
-<pinref part="IC2" gate="G$1" pin="GPB2"/>
+<pinref part="IC1" gate="G$1" pin="GPB2"/>
 <wire x1="53.34" y1="68.58" x2="58.42" y2="68.58" width="0.1524" layer="91"/>
 <wire x1="58.42" y1="68.58" x2="58.42" y2="71.12" width="0.1524" layer="91"/>
@@
 <pinref part="MCU" gate="A" pin="13"/>
 <wire x1="127" y1="68.58" x2="106.68" y2="68.58" width="0.1524" layer="91"/>
-<pinref part="IC2" gate="G$1" pin="GPB3"/>
+<pinref part="IC1" gate="G$1" pin="GPB3"/>
 <wire x1="106.68" y1="68.58" x2="104.14" y2="68.58" width="0.1524" layer="91"/>
 <wire x1="53.34" y1="66.04" x2="60.96" y2="66.04" width="0.1524" layer="91"/>
@@
 <segment>
 <pinref part="MCU" gate="A" pin="14"/>
-<pinref part="IC2" gate="G$1" pin="GPB4"/>
+<pinref part="IC1" gate="G$1" pin="GPB4"/>
 <wire x1="53.34" y1="63.5" x2="63.5" y2="63.5" width="0.1524" layer="91"/>
 <wire x1="63.5" y1="63.5" x2="63.5" y2="66.04" width="0.1524" layer="91"/>
@@
 <segment>
 <pinref part="MCU" gate="A" pin="15"/>
-<pinref part="IC2" gate="G$1" pin="GPB5"/>
+<pinref part="IC1" gate="G$1" pin="GPB5"/>
 <wire x1="53.34" y1="60.96" x2="66.04" y2="60.96" width="0.1524" layer="91"/>
 <wire x1="66.04" y1="60.96" x2="66.04" y2="63.5" width="0.1524" layer="91"/>
@@
 <pinref part="MCU" gate="A" pin="16"/>
 <wire x1="127" y1="60.96" x2="68.58" y2="60.96" width="0.1524" layer="91"/>
-<pinref part="IC2" gate="G$1" pin="GPB6"/>
+<pinref part="IC1" gate="G$1" pin="GPB6"/>
 <wire x1="53.34" y1="58.42" x2="68.58" y2="58.42" width="0.1524" layer="91"/>
 <wire x1="68.58" y1="58.42" x2="68.58" y2="60.96" width="0.1524" layer="91"/>
@@
 <pinref part="MCU" gate="A" pin="17"/>
 <wire x1="127" y1="58.42" x2="71.12" y2="58.42" width="0.1524" layer="91"/>
-<pinref part="IC2" gate="G$1" pin="GPB7"/>
+<pinref part="IC1" gate="G$1" pin="GPB7"/>
 <wire x1="53.34" y1="55.88" x2="71.12" y2="55.88" width="0.1524" layer="91"/>
 <wire x1="71.12" y1="55.88" x2="71.12" y2="58.42" width="0.1524" layer="91"/>
