File: eagle-boards/trinket-m0/trinket-mcp23016.brd (EAGLE design)
At the start: 53.6 x 34 mm, 10 parts, among them IC1 MCP23016P, Q1 BC547

Commit message: Update the capacitor to match the 8051 board.
Parts:
- C1: device rcl:C025-030X050 -> rcl:C025-025X050
Changed lines of the file:
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@@
 <attribute name="VALUE" x="47.2186" y="11.6586" size="0.9906" layer="21" ratio="10" rot="R270"/>
 </element>
-<element name="C1" library="rcl" library_urn="urn:adsk.eagle:library:334" package="C025-030X050" package3d_urn="urn:adsk.eagle:package:23631/1" value="33pF" x="12.7" y="11.43" smashed="yes" rot="R180">
+<element name="C1" library="rcl" library_urn="urn:adsk.eagle:library:334" package="C025-025X050" package3d_urn="urn:adsk.eagle:package:23629/2" value="33pF" x="12.7" y="11.43" smashed="yes" rot="R180">
 <attribute name="NAME" x="9.144" y="13.335" size="1.27" layer="25" ratio="10"/>
-<attribute name="POPULARITY" value="14" x="12.7" y="11.43" size="1.778" layer="27" rot="R180" display="off"/>
+<attribute name="POPULARITY" value="65" x="12.7" y="11.43" size="1.778" layer="27" rot="R180" display="off"/>
 <attribute name="SPICEPREFIX" value="C" x="12.7" y="11.43" size="1.778" layer="27" rot="R180" display="off"/>
 <attribute name="VALUE" x="11.938" y="13.335" size="1.27" layer="21" ratio="10"/>
