File: eagle-boards/trinket-m0/trinket-mcp23016.sch (EAGLE design)
At the start: 10 parts, among them IC1 MCP23016P, Q1 BC547

Commit message: Update the capacitor to match the 8051 board.
Parts:
- C1: device rcl:C-EU025-030X050 -> rcl:C-EU025-025X050
Changed lines of the file:
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@@
 <part name="+3V4" library="supply1" library_urn="urn:adsk.eagle:library:371" deviceset="+3V3" device=""/>
 <part name="R4" library="rcl" library_urn="urn:adsk.eagle:library:334" deviceset="R-EU_" device="0207/10" package3d_urn="urn:adsk.eagle:package:23491/2" value="3.9k"/>
-<part name="C1" library="rcl" library_urn="urn:adsk.eagle:library:334" deviceset="C-EU" device="025-030X050" package3d_urn="urn:adsk.eagle:package:23631/1" value="33pF"/>
+<part name="C1" library="rcl" library_urn="urn:adsk.eagle:library:334" deviceset="C-EU" device="025-025X050" package3d_urn="urn:adsk.eagle:package:23629/2" value="33pF"/>
 </parts>
 <sheets>
